File: hardware/ledstrip/ledstrip.kicad_sch (KiCad schematic)
At the start: 20 parts, among them J1 Conn_ARM_JTAG_SWD_10, J2 USB_C_Receptacle_USB2.0_16P, U1 STM32G030K6Tx, U2 CP2102N-A02-GQFN20, U4 USBLC6-2SC6

Commit message: Fix ERC and DRC errors.
Use a custom copy of USB-C in project library to avoid having a version
mismatch with CI.
Fix QFN-20-1EP_3x4mm_P0.5mm_EP1.65x2.65mm_ThermalVias  mismatch pins.
Fix ERC errors.
Parts:
- J2: footprint Connector_USB:USB_C_Receptacle_GCT_USB4105-xx-A_16P_TopMnt_Horizontal -> ledstrip:USB_C_Receptacle_GCT_USB4105-xx-A_16P_TopMnt_Horizontal_PROJECT_COPY
Changed lines of the file:
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@@
-	)
-	(junction
-		(at 157.48 119.38)
-		(diameter 0)
-		(color 0 0 0 0)
 	)
 	(junction
@@
 	(wire
 		(pts
-			(xy 157.48 118.11) (xy 157.48 119.38)
+			(xy 157.48 118.11) (xy 157.48 123.19)
 		)
 		(stroke
@@
 		(pts
 			(xy 204.47 120.65) (xy 259.08 120.65)
-		)
-		(stroke
-			(width 0)
-			(type default)
-		)
-	)
-	(wire
-		(pts
-			(xy 157.48 119.38) (xy 157.48 123.19)
 		)
 		(stroke
@@
 			)
 		)
-		(property "Footprint" "Connector_USB:USB_C_Receptacle_GCT_USB4105-xx-A_16P_TopMnt_Horizontal"
+		(property "Footprint" "ledstrip:USB_C_Receptacle_GCT_USB4105-xx-A_16P_TopMnt_Horizontal_PROJECT_COPY"
 			(at 35.56 143.51 0)
 			(effects
@@
 					(unit 1)
 				)
-			)
-		)
-	)
-	(symbol
-		(lib_id "power:PWR_FLAG")
-		(at 157.48 119.38 270)
-		(unit 1)
-		(exclude_from_sim no)
-		(in_bom yes)
-		(on_board yes)
-		(dnp no)
-		(property "Reference" "#FLG05"
-			(at 159.385 119.38 0)
-			(effects
-				(font
-					(size 1.27 1.27)
-				)
-				(hide yes)
-			)
-		)
-		(property "Value" "PWR_FLAG"
-			(at 162.56 121.666 90)
-			(effects
-				(font
-					(size 1.27 1.27)
-				)
-			)
-		)
-		(property "Footprint" ""
-			(at 157.48 119.38 0)
-			(effects
-				(font
-					(size 1.27 1.27)
-				)
-				(hide yes)
-			)
-		)
-		(property "Datasheet" "~"
-			(at 157.48 119.38 0)
-			(effects
-				(font
-					(size 1.27 1.27)
-				)
-				(hide yes)
-			)
-		)
-		(property "Description" "Special symbol for telling ERC where power comes from"
-			(at 157.48 119.38 0)
-			(effects
-				(font
-					(size 1.27 1.27)
-				)
-				(hide yes)
-			)
-		)
-		(pin "1"
-		)
-		(instances
-			(project "ledstrip"
-				(path "/dcb997ee-94c4-4df2-ba22-0e091735ddd7"
-					(reference "#FLG05")
-					(unit 1)
-				)
