File: hardware/ledstrip/ledstrip.kicad_sch (KiCad schematic)
At the start: 20 parts, among them J1 Conn_ARM_JTAG_SWD_10, J2 USB_C_Receptacle_USB2.0_16P, U1 STM32G030K6Tx, U2 CP2102N-A02-GQFN20, U4 USBLC6-2SC6

Commit message: Add a part number for USB port
Parts:
- J2: Disributor Link 1 (none) -> https://www.mouser.fr/ProductDetail/GCT/USB4105-GF-A-060?qs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; MPN (none) -> USB4105-GF-A-060; Manufacturer (none) -> GCT
Changed lines of the file:
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@@
 			)
 		)
-		(property "Disributor Link 1" ""
+		(property "Disributor Link 1" "https://www.mouser.fr/ProductDetail/GCT/USB4105-GF-A-060?qs=QNEnbhJQKvY2mocwNJzgfA%3D%3D"
 			(at 31.75 143.51 0)
 			(effects
@@
 			)
 		)
-		(property "Ditributor Link 1" ""
+		(property "MPN" "USB4105-GF-A-060"
 			(at 31.75 143.51 0)
 			(effects
+				(font
+					(size 1.27 1.27)
+				)
+				(hide yes)
+			)
+		)
+		(property "Manufacturer" "GCT"
+			(at 31.75 143.51 0)
+			(effects

Commit message: Minor fixes
Parts:
- C1, C4: MPN (none) -> CL21A106KAYNNN; Manufacturer Part Number CL21A106KAYNNN -> (none)
- C2, C3, C5: MPN (none) -> CL10B104KA8VPJC; Manufacturer Part Number CL10B104KA8VPJC -> (none)
- J2: Disributor Link 1 https://www.mouser.fr/ProductDetail/GCT/USB4105-GF-A-060?qs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 -> (none); Distributor Link 1 (none) -> https://www.mouser.fr/ProductDetail/GCT/USB4105-GF-A-060?qs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
- R3, R32, R33, R34: MPN (none) -> MCU0805MD1002BP500; Manufacturer (none) -> Vishay
- U1: MPN (none) -> STM32G030K6T6; Manufacturer Part Number STM32G030K6T6 -> (none)
- U2: MPN (none) -> CP2102N-A02-GQFN20; Manufacturer Part Number CP2102N-A02-GQFN20 -> (none)

Commit message: Update schematics symbols fields for manufactrurer
Update BOM fields.
Parts:
- R38: MPN (none) -> MCU0805MD1002BP500; Manufacturer (none) -> Vishay Beyschlag
- U4: MPN (none) -> USBLC6-2SC6; Manufacturer (none) -> STMicroelectronics

Commit message: Fix some symbols fields.
Parts:
- J1: Distributor Link 1 (none) -> https://www.mouser.com/ProductDetail/Harwin/M50-3500542?qs=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; MPN (none) -> M50-3500542; Manufacturer (none) -> Harwin
Changed lines of the file:
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@@
 			)
 		)
-		(property "Disributor Link 1" ""
+		(property "Distributor Link 1" "https://www.mouser.com/ProductDetail/Harwin/M50-3500542?qs=9fQaSFfsqsyXI0P9tFOVoQ%3D%3D"
 			(at 257.81 40.64 0)
 			(effects
@@
 			)
 		)
-		(property "Ditributor Link 1" ""
+		(property "Manufacturer" "Harwin"
 			(at 257.81 40.64 0)
 			(effects
@@
 			)
 		)
-		(property "Manufacturer Part Number" ""
+		(property "MPN" "M50-3500542"
 			(at 257.81 40.64 0)
 			(effects

Commit message: Fix ERC error
Parts:
- J1: Distributor Link 1 https://www.mouser.com/ProductDetail/Harwin/M50-3500542?qs=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 -> (none); MPN M50-3500542 -> (none); Manufacturer Harwin -> (none)
Changed lines of the file:
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@@
 			)
 		)
-		(property "Distributor Link 1" "https://www.mouser.com/ProductDetail/Harwin/M50-3500542?qs=9fQaSFfsqsyXI0P9tFOVoQ%3D%3D"
+		(property "Disributor Link 1" ""
 			(at 257.81 40.64 0)
 			(effects
@@
 			)
 		)
-		(property "Manufacturer" "Harwin"
+		(property "Ditributor Link 1" ""
 			(at 257.81 40.64 0)
 			(effects
@@
 			)
 		)
-		(property "MPN" "M50-3500542"
+		(property "Manufacturer Part Number" ""
 			(at 257.81 40.64 0)
 			(effects

Commit message: Normalize Vishay manufacturer (delete sub-brand)
Parts:
- R38: Manufacturer Vishay Beyschlag -> Vishay
Changed lines of the file:
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@@
 			)
 		)
-		(property "Manufacturer" "Vishay Beyschlag"
+		(property "Manufacturer" "Vishay"
 			(at 107.95 24.13 0)
 			(effects
