File: hardware/ledstrip/leds.kicad_sch (KiCad schematic)
At the start: 5 parts, among them J5 Ledstrip connector, Q1 Q_NMOS, Q11 Q_NMOS, Q2 Q_NMOS, Q3 Q_NMOS

Commit message: Update schematics symbols fields for manufactrurer
Update BOM fields.
Parts:
- Q1, Q11, Q2, Q3: MPN (none) -> IRL3705NPBF; Manufacturer (none) -> Infineon Technologies
Changed lines of the file:
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@@
+			)
+		)
+		(property "Manufacturer" "Infineon Technologies"
+			(at 161.29 109.22 0)
+			(effects
+				(font
+					(size 1.27 1.27)
+				)
+				(hide yes)
+			)
+		)
+		(property "MPN" "IRL3705NPBF"
+			(at 161.29 109.22 0)
+			(effects
+				(font
+					(size 1.27 1.27)
+				)
+				(hide yes)
 			)
 		)
 		(property "Distributor Link 2" "https://www.digikey.fr/fr/products/detail/infineon-technologies/IRL3705NPBF/812272?srsltid=AfmBOoooeDWkDS-ehnbFZ027sJbqecXx9GdmwNsCp8G_IMCaE9HrNfFl"
+			(at 161.29 109.22 0)
+			(effects
+				(font
+					(size 1.27 1.27)
+				)
+				(hide yes)
+			)
+		)
+		(property "Disributor Link 1" ""
+			(at 161.29 109.22 0)
+			(effects
+				(font
+					(size 1.27 1.27)
+				)
+				(hide yes)
+			)
+		)
+		(property "Ditributor Link 1" ""
+			(at 161.29 109.22 0)
+			(effects
+				(font
+					(size 1.27 1.27)
+				)
+				(hide yes)
+			)
+		)
+		(property "Manufacturer Part Number" ""
 			(at 161.29 109.22 0)
 			(effects
@@
 			)
 		)
+		(property "Manufacturer" "Infineon Technologies"
+			(at 146.05 109.22 0)
+			(effects
+				(font
+					(size 1.27 1.27)
+				)
+				(hide yes)
+			)
+		)
+		(property "MPN" "IRL3705NPBF"
+			(at 146.05 109.22 0)
+			(effects
+				(font
+					(size 1.27 1.27)
+				)
+				(hide yes)
+			)
+		)
 		(property "Distributor Link 2" "https://www.digikey.fr/fr/products/detail/infineon-technologies/IRL3705NPBF/812272?srsltid=AfmBOoooeDWkDS-ehnbFZ027sJbqecXx9GdmwNsCp8G_IMCaE9HrNfFl"
+			(at 146.05 109.22 0)
+			(effects
+				(font
+					(size 1.27 1.27)
+				)
+				(hide yes)
+			)
+		)
+		(property "Disributor Link 1" ""
+			(at 146.05 109.22 0)
+			(effects
+				(font
+					(size 1.27 1.27)
+				)
+				(hide yes)
+			)
+		)
+		(property "Ditributor Link 1" ""
+			(at 146.05 109.22 0)
+			(effects
+				(font
+					(size 1.27 1.27)
+				)
+				(hide yes)
+			)
+		)
+		(property "Manufacturer Part Number" ""
 			(at 146.05 109.22 0)
 			(effects
@@
 			)
 		)
+		(property "Manufacturer" "Infineon Technologies"
+			(at 114.3 109.22 0)
+			(effects
+				(font
+					(size 1.27 1.27)
+				)
+				(hide yes)
+			)
+		)
+		(property "MPN" "IRL3705NPBF"
+			(at 114.3 109.22 0)
+			(effects
+				(font
+					(size 1.27 1.27)
+				)
+				(hide yes)
+			)
+		)
 		(property "Distributor Link 2" "https://www.digikey.fr/fr/products/detail/infineon-technologies/IRL3705NPBF/812272?srsltid=AfmBOoooeDWkDS-ehnbFZ027sJbqecXx9GdmwNsCp8G_IMCaE9HrNfFl"
+			(at 114.3 109.22 0)
+			(effects
+				(font
+					(size 1.27 1.27)
+				)
+				(hide yes)
+			)
+		)
+		(property "Disributor Link 1" ""
+			(at 114.3 109.22 0)
+			(effects
+				(font
+					(size 1.27 1.27)
+				)
+				(hide yes)
+			)
+		)
+		(property "Ditributor Link 1" ""
+			(at 114.3 109.22 0)
+			(effects
+				(font
+					(size 1.27 1.27)
+				)
+				(hide yes)
+			)
+		)
+		(property "Manufacturer Part Number" ""
 			(at 114.3 109.22 0)
 			(effects
@@
 			)
 		)
+		(property "Manufacturer" "Infineon Technologies"
+			(at 130.81 109.22 0)
+			(effects
+				(font
+					(size 1.27 1.27)
+				)
+				(hide yes)
+			)
+		)
+		(property "MPN" "IRL3705NPBF"
+			(at 130.81 109.22 0)
+			(effects
+				(font
+					(size 1.27 1.27)
+				)
+				(hide yes)
+			)
+		)
 		(property "Distributor Link 2" "https://www.digikey.fr/fr/products/detail/infineon-technologies/IRL3705NPBF/812272?srsltid=AfmBOoooeDWkDS-ehnbFZ027sJbqecXx9GdmwNsCp8G_IMCaE9HrNfFl"
+			(at 130.81 109.22 0)
+			(effects
+				(font
+					(size 1.27 1.27)
+				)
+				(hide yes)
+			)
+		)
+		(property "Disributor Link 1" ""
+			(at 130.81 109.22 0)
+			(effects
+				(font
+					(size 1.27 1.27)
+				)
+				(hide yes)
+			)
+		)
+		(property "Ditributor Link 1" ""
+			(at 130.81 109.22 0)
+			(effects
+				(font
+					(size 1.27 1.27)
+				)
+				(hide yes)
+			)
+		)
+		(property "Manufacturer Part Number" ""
 			(at 130.81 109.22 0)
 			(effects
@@
 			(effects
 				(font
+					(size 1.27 1.27)
+				)
+				(hide yes)
+			)
+		)
+		(property "Disributor Link 1" ""
+			(at 119.38 59.69 90)
+			(effects
+				(font
+					(size 1.27 1.27)
+				)
+				(hide yes)
+			)
+		)
+		(property "Ditributor Link 1" ""
+			(at 119.38 59.69 90)
+			(effects
+				(font
+					(size 1.27 1.27)
+				)
+				(hide yes)
+			)
+		)
+		(property "Manufacturer Part Number" ""
+			(at 119.38 59.69 90)
+			(effects
+				(font

Commit message: Fix some symbols fields.
Parts:
- J5: Distributor Link 1 (none) -> https://nl.mouser.com/ProductDetail/JST-Commercial/B5B-XH-A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; MPN (none) -> B5B-XH-A(LF)(SN); Manufacturer (none) -> JST
Changed lines of the file:
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@@
 			)
 		)
-		(property "Disributor Link 1" ""
+		(property "Distributor Link 1" "https://nl.mouser.com/ProductDetail/JST-Commercial/B5B-XH-ALFSN?qs=cdbOS8ANM9ApoXpxtybURg%3D%3D"
 			(at 119.38 59.69 90)
 			(effects
@@
 			)
 		)
-		(property "Ditributor Link 1" ""
+		(property "Manufacturer" "JST"
 			(at 119.38 59.69 90)
 			(effects
@@
 			)
 		)
-		(property "Manufacturer Part Number" ""
+		(property "MPN" "B5B-XH-A(LF)(SN)"
 			(at 119.38 59.69 90)
 			(effects

Commit message: Fix ERC error
Parts:
- J5: Distributor Link 1 https://nl.mouser.com/ProductDetail/JST-Commercial/B5B-XH-A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 -> (none); MPN B5B-XH-A(LF)(SN) -> (none); Manufacturer JST -> (none)
Changed lines of the file:
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@@
 			)
 		)
-		(property "Distributor Link 1" "https://nl.mouser.com/ProductDetail/JST-Commercial/B5B-XH-ALFSN?qs=cdbOS8ANM9ApoXpxtybURg%3D%3D"
+		(property "Disributor Link 1" ""
 			(at 119.38 59.69 90)
 			(effects
@@
 			)
 		)
-		(property "Manufacturer" "JST"
+		(property "Ditributor Link 1" ""
 			(at 119.38 59.69 90)
 			(effects
@@
 			)
 		)
-		(property "MPN" "B5B-XH-A(LF)(SN)"
+		(property "Manufacturer Part Number" ""
 			(at 119.38 59.69 90)
 			(effects
