File: hardware/ledstrip/power_switch.kicad_sch (KiCad schematic)
At the start: 9 parts, among them SW1 SW_SPST, U8 TPS25940

Commit message: Add a BOM preset and set it in CI.
Parts:
- R39: Disributor Link 1 https://www.mouser.fr/ProductDetail/Vishay/TNPW080516K7BEEN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 -> (none); Distributor Link 1 (none) -> https://www.mouser.fr/ProductDetail/Vishay/TNPW080516K7BEEN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
- R4, R42: Distributor Link 1 (none) -> https://www.mouser.fr/ProductDetail/Vishay/CRCW0805475KFHEA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; Ditributor Link 1 https://www.mouser.fr/ProductDetail/Vishay/CRCW0805475KFHEA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 -> (none)
Changed lines of the file:
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@@
+			)
+		)
+		(property "Disributor Link 1" ""
+			(at 93.98 90.17 90)
+			(effects
+				(font
+					(size 1.27 1.27)
+				)
+				(hide yes)
+			)
+		)
+		(property "Ditributor Link 1" ""
+			(at 93.98 90.17 90)
+			(effects
+				(font
+					(size 1.27 1.27)
+				)
+				(hide yes)
 			)
 		)
@@
 			)
 		)
+		(property "Disributor Link 1" ""
+			(at 198.12 128.27 0)
+			(effects
+				(font
+					(size 1.27 1.27)
+				)
+				(hide yes)
+			)
+		)
+		(property "Ditributor Link 1" ""
+			(at 198.12 128.27 0)
+			(effects
+				(font
+					(size 1.27 1.27)
+				)
+				(hide yes)
+			)
+		)
 		(pin "1"
 		)
@@
 			)
 		)
+		(property "Disributor Link 1" ""
+			(at 111.76 134.62 0)
+			(effects
+				(font
+					(size 1.27 1.27)
+				)
+				(hide yes)
+			)
+		)
+		(property "Ditributor Link 1" ""
+			(at 111.76 134.62 0)
+			(effects
+				(font
+					(size 1.27 1.27)
+				)
+				(hide yes)
+			)
+		)
 		(pin "1"
 		)
@@
 			)
 		)
+		(property "Disributor Link 1" ""
+			(at 93.98 130.81 0)
+			(effects
+				(font
+					(size 1.27 1.27)
+				)
+				(hide yes)
+			)
+		)
+		(property "Ditributor Link 1" ""
+			(at 93.98 130.81 0)
+			(effects
+				(font
+					(size 1.27 1.27)
+				)
+				(hide yes)
+			)
+		)
 		(pin "2"
 		)
@@
 			)
 		)
+		(property "Disributor Link 1" ""
+			(at 125.73 106.68 0)
+			(effects
+				(font
+					(size 1.27 1.27)
+				)
+				(hide yes)
+			)
+		)
+		(property "Ditributor Link 1" ""
+			(at 125.73 106.68 0)
+			(effects
+				(font
+					(size 1.27 1.27)
+				)
+				(hide yes)
+			)
+		)
 		(pin "17"
 		)
@@
 			)
 		)
-		(property "Ditributor Link 1" "https://www.mouser.fr/ProductDetail/Vishay/CRCW0805475KFHEAP?qs=sGAEpiMZZMtlubZbdhIBIHs6lnEEKI8AuptDsuU1zU0%3D"
+		(property "Distributor Link 1" "https://www.mouser.fr/ProductDetail/Vishay/CRCW0805475KFHEAP?qs=sGAEpiMZZMtlubZbdhIBIHs6lnEEKI8AuptDsuU1zU0%3D"
+			(at 176.53 116.84 0)
+			(effects
+				(font
+					(size 1.27 1.27)
+				)
+				(hide yes)
+			)
+		)
+		(property "Disributor Link 1" ""
+			(at 176.53 116.84 0)
+			(effects
+				(font
+					(size 1.27 1.27)
+				)
+				(hide yes)
+			)
+		)
+		(property "Ditributor Link 1" ""
 			(at 176.53 116.84 0)
 			(effects
@@
 			)
 		)
-		(property "Ditributor Link 1" "https://www.mouser.fr/ProductDetail/Vishay/CRCW0805475KFHEAP?qs=sGAEpiMZZMtlubZbdhIBIHs6lnEEKI8AuptDsuU1zU0%3D"
+		(property "Distributor Link 1" "https://www.mouser.fr/ProductDetail/Vishay/CRCW0805475KFHEAP?qs=sGAEpiMZZMtlubZbdhIBIHs6lnEEKI8AuptDsuU1zU0%3D"
+			(at 93.98 102.87 0)
+			(effects
+				(font
+					(size 1.27 1.27)
+				)
+				(hide yes)
+			)
+		)
+		(property "Disributor Link 1" ""
+			(at 93.98 102.87 0)
+			(effects
+				(font
+					(size 1.27 1.27)
+				)
+				(hide yes)
+			)
+		)
+		(property "Ditributor Link 1" ""
 			(at 93.98 102.87 0)
 			(effects
@@
 			)
 		)
-		(property "Disributor Link 1" "https://www.mouser.fr/ProductDetail/Vishay/TNPW080516K7BEEN?qs=IW9Tsl75qsWQuKtQCpvGZQ%3D%3D"
+		(property "Distributor Link 1" "https://www.mouser.fr/ProductDetail/Vishay/TNPW080516K7BEEN?qs=IW9Tsl75qsWQuKtQCpvGZQ%3D%3D"
+			(at 93.98 115.57 0)
+			(effects
+				(font
+					(size 1.27 1.27)
+				)
+				(hide yes)
+			)
+		)
+		(property "Disributor Link 1" ""
+			(at 93.98 115.57 0)
+			(effects
+				(font
+					(size 1.27 1.27)
+				)
+				(hide yes)
+			)
+		)
+		(property "Ditributor Link 1" ""
 			(at 93.98 115.57 0)
 			(effects
@@
 			(at 170.18 137.16 0)
 			(effects
+				(font
+					(size 1.27 1.27)
+				)
+				(hide yes)
+			)
+		)
+		(property "Disributor Link 1" ""
+			(at 170.18 137.16 0)
+			(effects
+				(font
+					(size 1.27 1.27)
+				)
+				(hide yes)
+			)
+		)
+		(property "Ditributor Link 1" ""
+			(at 170.18 137.16 0)
+			(effects

Commit message: Update schematics symbols fields for manufactrurer
Update BOM fields.
Parts:
- C35: MPN (none) -> MLASE32MAB5107MPNA01; Manufacturer (none) -> TAIYO YUDEN
- C36: MPN (none) -> GRT033R61A152KE01D; Manufacturer (none) -> Murata Electronics
- R36: MPN (none) -> TNPW080517K8BETY; Manufacturer (none) -> Vishay
- R39: MPN (none) -> TNPW080516K7BEEN; Manufacturer (none) -> Vishay
- R4, R42: MPN (none) -> CRCW0805475KFHEAP; Manufacturer (none) -> Vishay
- R40: MPN (none) -> TNPW080531K2BEEN; Manufacturer (none) -> Vishay
- SW1: MPN (none) -> SW3001A; Manufacturer (none) -> NKK Switches

Commit message: Fix some symbols fields.
Parts:
- U8: Distributor Link 1 (none) -> https://www.mouser.fr/ProductDetail/Texas-Instruments/TPS25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; MPN (none) -> TPS25940ARVCR; Manufacturer (none) -> Texas Instruments
Changed lines of the file:
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@@
 			)
 		)
-		(property "Datasheet" "https://ds.yuden.co.jp/TYCOMPAS/or/download?pn=MLAST063SCG681JFNA01&fileType=CA"
+		(property "Datasheet" "https://ds.yuden.co.jp/TYCOMPAS/ap/detail?pn=MLASE32MAB5107MPNA01&u=M"
 			(at 198.12 128.27 0)
 			(effects
@@
 			)
 		)
-		(property "Disributor Link 1" ""
-			(at 125.73 106.68 0)
-			(effects
-				(font
-					(size 1.27 1.27)
-				)
-				(hide yes)
-			)
-		)
-		(property "Ditributor Link 1" ""
-			(at 125.73 106.68 0)
-			(effects
-				(font
-					(size 1.27 1.27)
-				)
-				(hide yes)
-			)
-		)
-		(property "Manufacturer Part Number" ""
-			(at 125.73 106.68 0)
-			(effects
+		(property "Distributor Link 1" "https://www.mouser.fr/ProductDetail/Texas-Instruments/TPS25940ARVCR?qs=1MXlzafEN38UtOFn%252BxDXYg%3D%3D"
+			(at 125.73 106.68 0)
+			(effects
+				(font
+					(size 1.27 1.27)
+				)
+				(hide yes)
+			)
+		)
+		(property "Manufacturer" "Texas Instruments"
+			(at 125.73 106.68 0)
+			(effects
+				(font
+					(size 1.27 1.27)
+				)
+				(hide yes)
+			)
+		)
+		(property "MPN" "TPS25940ARVCR"
+			(at 125.73 106.68 0)
+			(effects

Commit message: Fix ERC error
Parts:
- U8: Distributor Link 1 https://www.mouser.fr/ProductDetail/Texas-Instruments/TPS25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 -> (none); MPN TPS25940ARVCR -> (none); Manufacturer Texas Instruments -> (none)
Changed lines of the file:
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@@
 			)
 		)
-		(property "Datasheet" "https://ds.yuden.co.jp/TYCOMPAS/ap/detail?pn=MLASE32MAB5107MPNA01&u=M"
+		(property "Datasheet" "https://ds.yuden.co.jp/TYCOMPAS/or/download?pn=MLAST063SCG681JFNA01&fileType=CA"
 			(at 198.12 128.27 0)
 			(effects
@@
 			)
 		)
-		(property "Distributor Link 1" "https://www.mouser.fr/ProductDetail/Texas-Instruments/TPS25940ARVCR?qs=1MXlzafEN38UtOFn%252BxDXYg%3D%3D"
-			(at 125.73 106.68 0)
-			(effects
-				(font
-					(size 1.27 1.27)
-				)
-				(hide yes)
-			)
-		)
-		(property "Manufacturer" "Texas Instruments"
-			(at 125.73 106.68 0)
-			(effects
-				(font
-					(size 1.27 1.27)
-				)
-				(hide yes)
-			)
-		)
-		(property "MPN" "TPS25940ARVCR"
-			(at 125.73 106.68 0)
-			(effects
+		(property "Disributor Link 1" ""
+			(at 125.73 106.68 0)
+			(effects
+				(font
+					(size 1.27 1.27)
+				)
+				(hide yes)
+			)
+		)
+		(property "Ditributor Link 1" ""
+			(at 125.73 106.68 0)
+			(effects
+				(font
+					(size 1.27 1.27)
+				)
+				(hide yes)
+			)
+		)
+		(property "Manufacturer Part Number" ""
+			(at 125.73 106.68 0)
+			(effects
