File: hardware/ledstrip/batt.kicad_sch (KiCad schematic)
At the start: 51 parts, among them J4 BMS connectors, Q10 Q_PMOS, Q5 Q_NMOS, Q6 Q_NMOS, Q7 Q_NMOS, Q8 Q_NMOS, U5 BQ25703A, U7 TL431DBZ

Commit message: Minor fixes
Parts:
- C16, C18: MPN (none) -> CL10B104KA8VPJC; Manufacturer Part Number CL10B104KA8VPJC -> (none)
- C17, C26, C27, C28, C29, C30, C32: MPN (none) -> CL21A106KAYNNN; Manufacturer Part Number CL21A106KAYNNN -> (none)

Commit message: Update schematics symbols fields for manufactrurer
Update BOM fields.
Parts:
- C10: MPN (none) -> C0603C474J3RACTU; Manufacturer (none) -> KEMET
- C11, C12: MPN (none) -> 06031C333KAT2A; Manufacturer (none) -> KYOCERA AVX
- C13, C14: MPN (none) -> KGM15AR51V473KT; Manufacturer (none) -> KYOCERA AVX
- C15: MPN (none) -> 03028-BR103YKU-J; Manufacturer (none) -> Vishay Vitramon
- C19: MPN (none) -> KGQ15ACG2A330GT; Manufacturer (none) -> KYOCERA AVX
- C20: MPN (none) -> VJ0603Y182JXAAC; Manufacturer (none) -> Vishay Vitramon
- C21: MPN (none) -> 06031U150JAT2A; Manufacturer (none) -> KYOCERA AVX
- C22: MPN (none) -> VJ0603A681GXAAC; Manufacturer (none) -> Vishay Vitramon
- C31: MPN (none) -> 20TQC47MYF; Manufacturer (none) -> Panasonic
- C33: MPN (none) -> CL03A225MO5C65C; Manufacturer (none) -> Samsung Electro-Mechanics
- C34: MPN (none) -> AMK063AC6105MP-F; Manufacturer (none) -> TAIYO YUDEN
- L1: MPN (none) -> 74437356022; Manufacturer (none) -> Wurth Elektronik
- Q10: MPN (none) -> STL6P3LLH6; Manufacturer (none) -> STMicroelectronics
- Q5, Q6, Q7, Q8: MPN (none) -> CSD17551Q3A; Manufacturer (none) -> Texas Instruments
- R15: MPN (none) -> AC0805FR-071RL; Manufacturer (none) -> YAGEO
- R16, R21: MPN (none) -> WSLP0805R0100DEA; Manufacturer (none) -> Vishay Dale
- R17, R18: MPN (none) -> CRCW08054R99DKEAHP; Manufacturer (none) -> Vishay
- R19, R20: MPN (none) -> MCU0805MC1009FP500; Manufacturer (none) -> Vishay Beyschlag
- R22: MPN (none) -> CRCW080510R0JNEAHP; Manufacturer (none) -> Vishay
- R23, R27: MPN (none) -> RT0805BRB07100KL; Manufacturer (none) -> YAGEO
- R24: MPN (none) -> ERA-6ARB823V; Manufacturer (none) -> Panasonic
- R25: MPN (none) -> PHP00805E40R2BST1; Manufacturer (none) -> Vishay Thin Film
- R26, R29, R30: MPN (none) -> MCU0805MD1002BP500; Manufacturer (none) -> Vishay Beyschlag
- R28: MPN (none) -> CRCW0805107KFKEA; Manufacturer (none) -> Vishay
- R37: MPN (none) -> RCA06031K00FKEAHP; Manufacturer (none) -> Vishay Draloric
- U5: MPN (none) -> BQ25703ARSNR; Manufacturer (none) -> Texas Instruments
- U7: MPN (none) -> TL431AQDBZR; Manufacturer (none) -> Texas Instruments

Commit message: Fix some symbols fields.
Parts:
- J4: Distributor Link 1 (none) -> https://www.mouser.com/ProductDetail/Harwin/M20-9990246?qs=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; MPN (none) -> M20-9990246; Manufacturer (none) -> Harwin
Changed lines of the file:
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@@
 			)
 		)
-		(property "Datasheet" "https://www.yuden.co.jp/productdata/catalog/mlcc02_e.pdf"
+		(property "Datasheet" "https://ds.yuden.co.jp/TYCOMPAS/ap/detail?pn=MSASA063AC6105MFNA01&u=M"
 			(at 60.96 93.98 0)
 			(effects
@@
 			)
 		)
-		(property "Disributor Link 1" ""
+		(property "Distributor Link 1" "https://www.mouser.com/ProductDetail/Harwin/M20-9990246?qs=Jph8NoUxIfWjw4WmyRvzag%3D%3D"
 			(at 252.73 31.75 90)
 			(effects
@@
 			)
 		)
-		(property "Ditributor Link 1" ""
+		(property "Manufacturer" "Harwin"
 			(at 252.73 31.75 90)
 			(effects
@@
 			)
 		)
-		(property "Manufacturer Part Number" ""
+		(property "MPN" "M20-9990246"
 			(at 252.73 31.75 90)
 			(effects

Commit message: Fix ERC error
Parts:
- J4: Distributor Link 1 https://www.mouser.com/ProductDetail/Harwin/M20-9990246?qs=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 -> (none); MPN M20-9990246 -> (none); Manufacturer Harwin -> (none)
Changed lines of the file:
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@@
 			)
 		)
-		(property "Datasheet" "https://ds.yuden.co.jp/TYCOMPAS/ap/detail?pn=MSASA063AC6105MFNA01&u=M"
+		(property "Datasheet" "https://www.yuden.co.jp/productdata/catalog/mlcc02_e.pdf"
 			(at 60.96 93.98 0)
 			(effects
@@
 			)
 		)
-		(property "Distributor Link 1" "https://www.mouser.com/ProductDetail/Harwin/M20-9990246?qs=Jph8NoUxIfWjw4WmyRvzag%3D%3D"
+		(property "Disributor Link 1" ""
 			(at 252.73 31.75 90)
 			(effects
@@
 			)
 		)
-		(property "Manufacturer" "Harwin"
+		(property "Ditributor Link 1" ""
 			(at 252.73 31.75 90)
 			(effects
@@
 			)
 		)
-		(property "MPN" "M20-9990246"
+		(property "Manufacturer Part Number" ""
 			(at 252.73 31.75 90)
 			(effects

Commit message: Normalize Vishay manufacturer (delete sub-brand)
Parts:
- C15, C20, C22: Manufacturer Vishay Vitramon -> Vishay
- R16, R21: Manufacturer Vishay Dale -> Vishay
- R19, R20, R26, R29, R30: Manufacturer Vishay Beyschlag -> Vishay
- R25: Manufacturer Vishay Thin Film -> Vishay
- R37: Manufacturer Vishay Draloric -> Vishay
Changed lines of the file:
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@@
 			)
 		)
-		(property "Manufacturer" "Vishay Dale"
+		(property "Manufacturer" "Vishay"
 			(at 198.12 38.1 0)
 			(effects
@@
 			)
 		)
-		(property "Manufacturer" "Vishay Beyschlag"
+		(property "Manufacturer" "Vishay"
 			(at 151.13 191.77 0)
 			(effects
@@
 			)
 		)
-		(property "Manufacturer" "Vishay Vitramon"
+		(property "Manufacturer" "Vishay"
 			(at 114.3 34.29 90)
 			(effects
@@
 			)
 		)
-		(property "Manufacturer" "Vishay Vitramon"
+		(property "Manufacturer" "Vishay"
 			(at 52.07 146.05 90)
 			(effects
@@
 			)
 		)
-		(property "Manufacturer" "Vishay Beyschlag"
+		(property "Manufacturer" "Vishay"
 			(at 175.26 74.93 0)
 			(effects
@@
 			)
 		)
-		(property "Manufacturer" "Vishay Beyschlag"
+		(property "Manufacturer" "Vishay"
 			(at 104.14 163.83 0)
 			(effects
@@
 			)
 		)
-		(property "Manufacturer" "Vishay Beyschlag"
+		(property "Manufacturer" "Vishay"
 			(at 182.88 74.93 0)
 			(effects
@@
 			)
 		)
-		(property "Manufacturer" "Vishay Dale"
+		(property "Manufacturer" "Vishay"
 			(at 97.79 24.13 0)
 			(effects
@@
 			)
 		)
-		(property "Manufacturer" "Vishay Draloric"
+		(property "Manufacturer" "Vishay"
 			(at 43.18 55.88 90)
 			(effects
@@
 			)
 		)
-		(property "Manufacturer" "Vishay Thin Film"
+		(property "Manufacturer" "Vishay"
 			(at 67.31 146.05 0)
 			(effects
@@
 			)
 		)
-		(property "Manufacturer" "Vishay Vitramon"
+		(property "Manufacturer" "Vishay"
 			(at 52.07 152.4 90)
 			(effects
@@
 			)
 		)
-		(property "Manufacturer" "Vishay Beyschlag"
+		(property "Manufacturer" "Vishay"
 			(at 67.31 152.4 0)
 			(effects
