File: hardware/ledstrip/batt.kicad_sch (KiCad schematic)
At the start: 57 parts, among them J4 BMS connectors, Q10 Q_PMOS, Q5 Q_NMOS, Q6 Q_NMOS, Q7 Q_NMOS, Q8 Q_NMOS, U5 BQ25703A, U7 TL431DBZ

Commit message: Use exact MPN instead of "base" MPN for CL21A106KAYNNN(F)
Parts:
- C17, C26, C27, C28, C29, C30, C32: MPN CL21A106KAYNNN -> CL21A106KAYNNNF
Changed lines of the file:
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@@
 			)
 		)
-		(property "MPN" "CL21A106KAYNNN"
+		(property "MPN" "CL21A106KAYNNNF"
 			(at 193.04 20.32 0)
 			(effects
@@
 			)
 		)
-		(property "MPN" "CL21A106KAYNNN"
+		(property "MPN" "CL21A106KAYNNNF"
 			(at 223.52 20.32 0)
 			(effects
@@
 			)
 		)
-		(property "MPN" "CL21A106KAYNNN"
+		(property "MPN" "CL21A106KAYNNNF"
 			(at 213.36 20.32 0)
 			(effects
@@
 			)
 		)
-		(property "MPN" "CL21A106KAYNNN"
+		(property "MPN" "CL21A106KAYNNNF"
 			(at 233.68 20.32 0)
 			(effects
@@
 			)
 		)
-		(property "MPN" "CL21A106KAYNNN"
+		(property "MPN" "CL21A106KAYNNNF"
 			(at 203.2 20.32 0)
 			(effects
@@
 			)
 		)
-		(property "MPN" "CL21A106KAYNNN"
+		(property "MPN" "CL21A106KAYNNNF"
 			(at 242.57 44.45 0)
 			(effects
@@
 			)
 		)
-		(property "MPN" "CL21A106KAYNNN"
+		(property "MPN" "CL21A106KAYNNNF"
 			(at 182.88 20.32 0)
 			(effects
