File: hardware/ledstrip/pwr.kicad_sch (KiCad schematic)
At the start: 32 parts, among them J6 Header for STUSB4500 I2C, Q4 Q_PMOS, Q9 Q_PMOS, U6 STUSB4500QTR

Commit message: Start editing some trace.
Changed lines of the file:
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@@
 	(generator_version "9.0")
 	(paper "A4")
-	(text_box "Theses FETs should always be openned by STUSB4500. It provide protections against hot-plug stress."
+	(text_box "Theses FETs should be openned by STUSB4500. It provide protections against hot-plug stress."
 		(exclude_from_sim no)
 		(at 205.74 12.7 0)
@@
 		)
 	)
-	(text_box "STUSB4500 programmation :\nAlways let the VBUS go (POWER_ONLY_ABOVE_5V=0b)"
+	(text_box "STUSB4500 programmation :\nAlways let the VBUS go (POWER_ONLY_ABOVE_5V=0b)\nSo, if high power available (15V) take it, if not just let go."
 		(exclude_from_sim no)
 		(at 205.74 129.54 0)
-		(size 60.96 5.08)
+		(size 60.96 7.62)
 		(margins 0.9525 0.9525 0.9525 0.9525)
 		(stroke

Commit message: Minor fixes
Parts:
- C25: MPN (none) -> CL10B104KA8VPJC; Manufacturer Part Number CL10B104KA8VPJC -> (none)

Commit message: Update schematics symbols fields for manufactrurer
Update BOM fields.
Parts:
- C6, C7, C8, C9: MPN (none) -> 885012106022; Manufacturer (none) -> Wurth Elektronik
- D1: Distributor Link 1 https://www.st.com/resource/en/datasheet/esda20p50-1u1m.pdf -> https://www.mouser.com/ProductDetail/STMicroelectronics/ESD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; MPN (none) -> ESDA20P50-1U1M; Manufacturer (none) -> STMicroelectronics
- D2: MPN (none) -> BAT54JFILM; Manufacturer (none) -> STMicroelectronics
- D3, D4: MPN (none) -> ESDALC5-1BT2; Manufacturer (none) -> STMicroelectronics
- D6: MPN (none) -> SMAJ15AHM3_A-H; Manufacturer (none) -> Vishay General Semiconductor
- Q4, Q9: MPN (none) -> STL6P3LLH6; Manufacturer (none) -> STMicroelectronics
- R1: MPN (none) -> CRCW080510R0JNEAHP; Manufacturer (none) -> Vishay
- R10, R7, R8, R9: MPN (none) -> ERA-6ARW472V; Manufacturer (none) -> Panasonic
- R11, R13: MPN (none) -> RT0805BRB07100KL; Manufacturer (none) -> YAGEO
- R12, R6: MPN (none) -> RCA06031K00FKEAHP; Manufacturer (none) -> Vishay Draloric
- R14: MPN (none) -> MCU08050C2202FP500; Manufacturer (none) -> Vishay Beyschlag
- R2: MPN (none) -> WSLP0805R0100DEA; Manufacturer (none) -> Vishay Dale
- R35: MPN (none) -> RP0805CT-1000GN-96TR; Manufacturer (none) -> Vishay Barry Industries
- R5: MPN (none) -> SFR03EZPJ471; Manufacturer (none) -> ROHM Semiconductor

Commit message: Fix some symbols fields.
Parts:
- J6: Distributor Link 1 (none) -> https://www.mouser.com/ProductDetail/Harwin/M20-9990446?qs=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; MPN (none) -> M20-9990446; Manufacturer (none) -> Harwin
- U6: Distributor Link 1 (none) -> https://estore.st.com/en/stusb4500qtr-cpn.html; MPN (none) -> STUSB4500QTR; Manufacturer (none) -> STMicroelectronics
Changed lines of the file:
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@@
 			)
 		)
-		(property "Disributor Link 1" ""
+		(property "Distributor Link 1" "https://www.mouser.com/ProductDetail/Harwin/M20-9990446?qs=ulE8k0yEMYaW%252BOM7jiG6%252Bw%3D%3D"
 			(at 55.88 93.98 0)
 			(effects
@@
 			)
 		)
-		(property "Ditributor Link 1" ""
+		(property "Manufacturer" "Harwin"
 			(at 55.88 93.98 0)
 			(effects
@@
 			)
 		)
-		(property "Manufacturer Part Number" ""
+		(property "MPN" "M20-9990446"
 			(at 55.88 93.98 0)
 			(effects
@@
 			)
 		)
-		(property "Disributor Link 1" ""
+		(property "Distributor Link 1" "https://estore.st.com/en/stusb4500qtr-cpn.html"
 			(at 162.56 86.36 0)
 			(effects
@@
 			)
 		)
-		(property "Ditributor Link 1" ""
+		(property "Manufacturer" "STMicroelectronics"
 			(at 162.56 86.36 0)
 			(effects
@@
 			)
 		)
-		(property "Manufacturer Part Number" ""
+		(property "MPN" "STUSB4500QTR"
 			(at 162.56 86.36 0)
 			(effects

Commit message: Fix ERC error
Parts:
- J6: Distributor Link 1 https://www.mouser.com/ProductDetail/Harwin/M20-9990446?qs=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 -> (none); MPN M20-9990446 -> (none); Manufacturer Harwin -> (none)
- U6: Distributor Link 1 https://estore.st.com/en/stusb4500qtr-cpn.html -> (none); MPN STUSB4500QTR -> (none); Manufacturer STMicroelectronics -> (none)
Changed lines of the file:
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@@
 			)
 		)
-		(property "Distributor Link 1" "https://www.mouser.com/ProductDetail/Harwin/M20-9990446?qs=ulE8k0yEMYaW%252BOM7jiG6%252Bw%3D%3D"
+		(property "Disributor Link 1" ""
 			(at 55.88 93.98 0)
 			(effects
@@
 			)
 		)
-		(property "Manufacturer" "Harwin"
+		(property "Ditributor Link 1" ""
 			(at 55.88 93.98 0)
 			(effects
@@
 			)
 		)
-		(property "MPN" "M20-9990446"
+		(property "Manufacturer Part Number" ""
 			(at 55.88 93.98 0)
 			(effects
@@
 			)
 		)
-		(property "Distributor Link 1" "https://estore.st.com/en/stusb4500qtr-cpn.html"
+		(property "Disributor Link 1" ""
 			(at 162.56 86.36 0)
 			(effects
@@
 			)
 		)
-		(property "Manufacturer" "STMicroelectronics"
+		(property "Ditributor Link 1" ""
 			(at 162.56 86.36 0)
 			(effects
@@
 			)
 		)
-		(property "MPN" "STUSB4500QTR"
+		(property "Manufacturer Part Number" ""
 			(at 162.56 86.36 0)
 			(effects

Commit message: Normalize Vishay manufacturer (delete sub-brand)
Parts:
- D6: Manufacturer Vishay General Semiconductor -> Vishay
- R12, R6: Manufacturer Vishay Draloric -> Vishay
- R14: Manufacturer Vishay Beyschlag -> Vishay
- R2: Manufacturer Vishay Dale -> Vishay
- R35: Manufacturer Vishay Barry Industries -> Vishay
Changed lines of the file:
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@@
 			)
 		)
-		(property "Manufacturer" "Vishay Barry Industries"
+		(property "Manufacturer" "Vishay"
 			(at 243.84 63.5 0)
 			(effects
@@
 			)
 		)
-		(property "Manufacturer" "Vishay General Semiconductor"
+		(property "Manufacturer" "Vishay"
 			(at 33.02 53.34 0)
 			(effects
@@
 			)
 		)
-		(property "Manufacturer" "Vishay Draloric"
+		(property "Manufacturer" "Vishay"
 			(at 82.55 85.09 90)
 			(effects
@@
 			)
 		)
-		(property "Manufacturer" "Vishay Dale"
+		(property "Manufacturer" "Vishay"
 			(at 44.45 22.86 0)
 			(effects
@@
 			)
 		)
-		(property "Manufacturer" "Vishay Beyschlag"
+		(property "Manufacturer" "Vishay"
 			(at 213.36 71.12 90)
 			(effects
@@
 			)
 		)
-		(property "Manufacturer" "Vishay Draloric"
+		(property "Manufacturer" "Vishay"
 			(at 224.79 88.9 90)
 			(effects
