File: hardware/ledstrip/pwr.kicad_sch (KiCad schematic)
At the start: 32 parts, among them J6 Header for STUSB4500 I2C, Q4 Q_PMOS, Q9 Q_PMOS, U6 STUSB4500QTR

Commit message: Fix a wrong capa and add MPN and stuff to STUSB4500
Parts:
- U6: Distributor Link 1 (none) -> https://www.mouser.com/ProductDetail/STMicroelectronics/STU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; Distributor Link 2 (none) -> https://www.digikey.fr/fr/products/detail/stmicroelectronic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; MPN (none) -> STUSB4500QTR; Manufacturer (none) -> STMicroelectronics
Changed lines of the file:
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@@
+			)
+		)
+		(property "Distributor Link 1" "https://www.mouser.com/ProductDetail/STMicroelectronics/STUSB4500QTR?qs=wUXugUrL1qyQbYMSzG1ujg%3D%3D&srsltid=AfmBOoqdJjWWB32R9DlfzH-bq0KiDhRy28r8GjITeKYE_sP4LKbWOqok"
+			(at 162.56 86.36 0)
+			(effects
+				(font
+					(size 1.27 1.27)
+				)
+				(hide yes)
+			)
+		)
+		(property "Distributor Link 2" "https://www.digikey.fr/fr/products/detail/stmicroelectronics/STUSB4500QTR/9092189?srsltid=AfmBOopQKGGuVsmmPkwv5fl12wAqcQkAnjHQZQxBTBIzbqYHhmdax9Te"
+			(at 162.56 86.36 0)
+			(effects
+				(font
+					(size 1.27 1.27)
+				)
+				(hide yes)
+			)
+		)
+		(property "Manufacturer" "STMicroelectronics"
+			(at 162.56 86.36 0)
+			(effects
+				(font
+					(size 1.27 1.27)
+				)
+				(hide yes)
+			)
+		)
+		(property "MPN" "STUSB4500QTR"
+			(at 162.56 86.36 0)
+			(effects
+				(font
+					(size 1.27 1.27)
+				)
+				(hide yes)
 			)
 		)

Commit message: Improve BOM: exclude uneeded parts, add some columns.
Parts:
- J6, TP1, TP2, TP3, TP4, TP5: now left out of the parts list

Commit message: Mark through-hole component "Do not place" in schematics.
Parts:
- J6: now not fitted
Changed lines of the file:
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@@
 		(in_bom no)
 		(on_board yes)
-		(dnp no)
+		(dnp yes)
 		(property "Reference" "J6"
 			(at 53.34 90.424 0)
@@
 			(at 55.88 93.98 0)
 			(effects
-				(font
-					(size 1.27 1.27)
-				)
-				(hide yes)
-			)
-		)
-		(property "Disributor Link 1" ""
-			(at 55.88 93.98 0)
-			(effects
-				(font
-					(size 1.27 1.27)
-				)
-				(hide yes)
-			)
-		)
-		(property "Ditributor Link 1" ""
-			(at 55.88 93.98 0)
-			(effects
-				(font
-					(size 1.27 1.27)
-				)
-				(hide yes)
-			)
-		)
-		(property "Manufacturer Part Number" ""
-			(at 55.88 93.98 0)
-			(effects

Commit message: Fix wrong footprint (C_0603 instead of R_0603)
Parts:
- R12, R5, R6: footprint Capacitor_SMD:C_0603_1608Metric -> Resistor_SMD:R_0603_1608Metric
Changed lines of the file:
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@@
 			)
 		)
-		(property "Footprint" "Capacitor_SMD:C_0603_1608Metric"
+		(property "Footprint" "Resistor_SMD:R_0603_1608Metric"
 			(at 69.85 86.868 90)
 			(effects
@@
 			)
 		)
-		(property "Footprint" "Capacitor_SMD:C_0603_1608Metric"
+		(property "Footprint" "Resistor_SMD:R_0603_1608Metric"
 			(at 82.55 86.868 90)
 			(effects
@@
 			)
 		)
-		(property "Footprint" "Capacitor_SMD:C_0603_1608Metric"
+		(property "Footprint" "Resistor_SMD:R_0603_1608Metric"
 			(at 224.79 90.678 90)
 			(effects
