File: hardware/ledstrip/pwr.kicad_sch (KiCad schematic)
At the start: 32 parts, among them J6 Header for STUSB4500 I2C, Q4 Q_PMOS, Q9 Q_PMOS, U6 STUSB4500QTR

Commit message: Update D1 with ST's replacement part.
Parts:
- D1: Distributor Link 1 https://www.mouser.com/ProductDetail/STMicroelectronics/ESD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 -> https://www.mouser.com/en/ProductDetail/STMicroelectronics/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; MPN ESDA20P50-1U1M -> ESDA25P35-1U1M; Manufacturer Part Number (none) -> ESDA25P35-1U1M
Changed lines of the file:
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@@
 			)
 		)
-		(property "Datasheet" "https://www.st.com/resource/en/datasheet/esda20p50-1u1m.pdf"
+		(property "Datasheet" "https://www.st.com/resource/en/datasheet/esda25p35-1u1m.pdf"
 			(at 260.35 53.34 0)
 			(effects
@@
 			)
 		)
-		(property "Distributor Link 1" "https://www.mouser.com/ProductDetail/STMicroelectronics/ESDA20P50-1U1M?qs=5aG0NVq1C4xh7oI9x8u0Tw%3D%3D"
+		(property "Distributor Link 1" "https://www.mouser.com/en/ProductDetail/STMicroelectronics/ESDA25P35-1U1M?qs=aVyJF2WnouQUWqgNP85ZrA%3D%3D"
 			(at 260.35 53.34 0)
 			(effects
@@
 			)
 		)
-		(property "MPN" "ESDA20P50-1U1M"
+		(property "MPN" "ESDA25P35-1U1M"
 			(at 260.35 53.34 0)
 			(effects
@@
 			)
 		)
-		(property "Manufacturer Part Number" ""
+		(property "Manufacturer Part Number" "ESDA25P35-1U1M"
 			(at 260.35 53.34 90)
 			(effects
