File: hardware/ledstrip/buck.kicad_sch (KiCad schematic)
At the start: 6 parts, among them U3 TPS62162DSG

Commit message: Use exact MPN instead of "base" MPN for CL21A106KAYNNN(F)
Parts:
- C23: MPN CL21A106KAYNNN -> CL21A106KAYNNNF
Changed lines of the file:
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@@
 			)
 		)
-		(property "MPN" "CL21A106KAYNNN"
+		(property "MPN" "CL21A106KAYNNNF"
 			(at 90.17 85.09 0)
 			(effects
